File: spiralboard.kicad_sch (KiCad schematic)
At the start: 4 parts

Commit message: mouting hole vergrößert
Parts:
- H1: footprint MountingHole:MountingHole_4mm_Pad_TopBottom -> MountingHole:MountingHole_5.3mm_M5_Pad_TopBottom
Changed lines of the file:
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@@
       (effects (font (size 1.27 1.27)) (justify left))
     )
-    (property "Footprint" "MountingHole:MountingHole_4mm_Pad_TopBottom" (at 44.45 171.45 0)
+    (property "Footprint" "MountingHole:MountingHole_5.3mm_M5_Pad_TopBottom" (at 44.45 171.45 0)
       (effects (font (size 1.27 1.27)) hide)
     )

Commit message: Linearregler getauscht, schalter hinzugefügt
Other:
- company: (none) -> @casartar
Changed lines of the file:
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@@
     (date "2023-07-01")
     (rev "v1.0")
+    (company "@casartar")
   )
   (wire (pts (xy 109.22 43.18) (xy 104.14 43.18))
