File: ws2812.kicad_sch (KiCad schematic)
At the start: 64 parts

Commit message: Linearregler getauscht, schalter hinzugefügt
Other:
- company: (none) -> @casartar
Changed lines of the file:
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@@
     (title "Spiralboard")
     (date "2023-07-01")
+    (rev "v1.0")
+    (company "@casartar")
   )
   (no_connect (at 274.32 151.13))
