File: PCB/ws2812.kicad_sch (KiCad schematic)
At the start: 64 parts

Commit message: docu update, add schematic pdf, file updates
Parts:
- renumbered C16 to C1, C3 to C10, C20 to C11, C32 to C12, C4 to C13, C21 to C14, C5 to C15, C22 to C16, C6 to C17, C23 to C18, C7 to C19, C17 to C2, C24 to C20, C8 to C21, C25 to C22, C9 to C23, C26 to C24, C10 to C25, C27 to C26, C11 to C27, C12 to C29, C29 to C3, C13 to C30, C14 to C31, C15 to C32, C1 to C4, C18 to C5, C30 to C6, C2 to C7, C19 to C8, C31 to C9, D4 to D10, D14 to D11, D24 to D12, D5 to D13, D15 to D14, D25 to D15, D6 to D16, D16 to D17, D26 to D18, D7 to D19, D11 to D2, D17 to D20, D27 to D21, D8 to D22, D18 to D23, D28 to D24, D9 to D25, D19 to D26, D29 to D27, D31 to D28, D10 to D29, D21 to D3, D20 to D30, D30 to D31, D2 to D4, D12 to D5, D22 to D6, D3 to D7, D13 to D8, D23 to D9
